File: _autosave-FPGA-power-source.kicad_sch (KiCad schematic)
At the start: 34 parts, among them U1 TPS54325PWPR, U2 TPS54294PWP

Commit message: FPGA power source passes ERC
Parts:
- C1, C2, C3, C4, C5: footprint (none) -> Capacitor_SMD:C_0805_2012Metric
- L1, L2, L3: footprint (none) -> Inductor_SMD:L_0805_2012Metric
- R1, R2, R3, R4, R5, R6, R7, R8, R9: footprint (none) -> Resistor_SMD:R_0805_2012Metric
- U1: footprint TPS54325PWPR:IC_TPS27S100BPWPR -> TPS54325PWPR:PWP14_2P31X2P46
- U2: footprint PWP16_2P31X2P46 -> TPS54294PWP:PWP16_2P31X2P46
