File: TDT4295.kicad_sch (KiCad schematic)
At the start: 0 parts

Commit message: VGA design
Other:
- sheet 8bit vga out renamed 4bit vga out
Changed lines of the file:
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@@
 			(color 0 0 0 0.0000)
 		)
-		(property "Sheetname" "8bit vga out"
+		(property "Sheetname" "4bit vga out"
 			(at 67.31 14.5284 0)
 			(effects
