File: Full_schematic.kicad_sch (KiCad schematic)
At the start: 206 parts, among them IC1 XC7A100T-1FTG256C, J4 FFC3B11-40-T, J6 Conn_ST_STDC14, SW3 SW_DPST_x2, SW4 SW_DPST_x2, U10 MC14511BDG, U11 MC14511BDG, U12 MAN72A, U13 MC14511BDG, U14 MAN72A, U2 TPS54294PWP, U2 TPS54325PWPR, U3 SN74ALVC245PWR, U4 SN74ALVC245PWR, U5 MC14511BDG, U6 MAN72A, U7 STM32U545VETxQ, U8 2S7A_0518S1U, U9 MAN72A, Y1 ASCO, Y4 48MHz

Commit message: merge 7seg with sram
Parts:
- removed C40, C41: 100n, symbol Device:C
- removed C62: 1210, 2.2µF/100V, symbol Device:C
- removed IC1: XC7A100T-1FTG256C, BGA256C100P16X16_1700X1700X155, symbol XC7A100T-1FTG256C:XC7A100T-1FTG256C
- removed J1: ~, symbol FPGA_Debug:FPGA_debug
- removed J2: ~, symbol PMod:PMod j1
- removed J2: ~, symbol PMod:PMod_j2
- removed J4: FFC3B11-40-T, FFC3B11-40-T:GCT_FFC3B11-40-T, symbol FFC3B11-40-T:FFC3B11-40-T
- removed L6: 18uH, symbol Device:L
- removed R1, R3: 4.7k, symbol Device:R
- removed R13 (x2), R14 (x2), R15 (x2), R16, R17, R18, R19, R20, R21, R22, R23: 100K, symbol Device:R
- removed R2: 2.4k, symbol Device:R
- removed R30, R31: 100, symbol Device:R
- removed R32, R33, R34, R35, R39, R40, R41, R42, R46, R47, R48, R49: 536, symbol Device:R
- removed R36, R37, R38, R43, R44, R45, R50, R51, R52: 270, symbol Device:R
- removed R4, R5: 10k, symbol Device:R
- removed R6: 330, symbol Device:R
- removed U1: ~, symbol S25FL127S:S25FL127S
- removed U3, U4: SN74ALVC245PWR, PW20, symbol 2025-09-12_09-11-34:SN74ALVC245PWR
- removed U8: 2S7A_0518S1U, SIP4_2S7A_GAP, symbol 2S7A_0518S1U:2S7A_0518S1U
- removed Y1: ASCO, Oscillator:Oscillator_SMD_Abracon_ASCO-4Pin_1.6x1.2mm, symbol Oscillator:ASCO
- added C132, C141: 100n, symbol Device:C
- added C144: 1210, 2.2µF/100V, symbol Device:C
- added IC2: XC7A100T-1FTG256C, BGA256C100P16X16_1700X1700X155, symbol XC7A100T-1FTG256C:XC7A100T-1FTG256C
- added J5: ~, symbol FPGA_Debug:FPGA_debug
- added J7: FFC3B11-40-T, FFC3B11-40-T:GCT_FFC3B11-40-T, symbol FFC3B11-40-T:FFC3B11-40-T
- added L11: 18uH, symbol Device:L
- added R100, R102, R104, R106, R107, R109, R111, R113, R116, R118, R120, R122: 536, symbol Device:R
- added R101, R103, R105, R108, R110, R112, R117, R119, R121: 270, symbol Device:R
- added R114, R115: 100, symbol Device:R
- added R123, R125: 4.7k, symbol Device:R
- added R124: 2.4k, symbol Device:R
- added R126, R127: 10k, symbol Device:R
- added R94: 330, symbol Device:R
- added U15, U19: ~, symbol SRAM:SRAM
- added U18, U20: SN74ALVC245PWR, PW20, symbol 2025-09-12_09-11-34:SN74ALVC245PWR
- added U21: ~, symbol S25FL127S:S25FL127S
- added U22: 2S7A_0518S1U, SIP4_2S7A_GAP, symbol 2S7A_0518S1U:2S7A_0518S1U
- added Y2: ASCO, Oscillator:Oscillator_SMD_Abracon_ASCO-4Pin_1.6x1.2mm, symbol Oscillator:ASCO
Connections:
- net +1V0: now also IC2.E10 (VCCBRAM_1), IC2.F11 (VCCBRAM_2), IC2.F7 (VCCINT_1), IC2.F9 (VCCINT_2), IC2.G6 (VCCINT_3), IC2.H9 (VCCINT_4), IC2.J6 (VCCINT_5), IC2.L8 (VCCINT_7)
- net +1V8: now also IC2.G10 (VCCAUX_1), IC2.G8 (VCCADC_0), IC2.J10 (VCCAUX_2), IC2.K11 (VCCAUX_3), IC2.L10 (VCCAUX_4)
- net +3.3V: now also J7.4, U18.1 (DIR), U18.20 (VCC), U20.1 (DIR), U20.20 (VCC)
- net +3V3: now also C132.1, C141.1, IC2.A16 (VCCO_15_1), IC2.B13 (VCCO_15_2), IC2.C10 (VCCO_15_3), IC2.E14 (VCCO_15_4), IC2.H15 (VCCO_15_5), IC2.J12 (VCCO_15_6), IC2.L16 (VCCO_14_1), IC2.L6 (VCCO_0), IC2.M13 (VCCO_14_2), IC2.N10 (VCCO_14_3), IC2.P7 (VCCO_14_4), IC2.R14 (VCCO_14_5), IC2.T11 (VCCO_14_6), J5.2, R123.1, R124.1, R125.1, R126.1, R127.1, R94.1, U21.8 (VCC), Y2.1 (Tri-State), Y2.4 (VDD)
- net +5V: now also C132.2, C141.2, C144.1, C144.2, IC2.A1 (GND_1), IC2.A11 (GND_2), IC2.B8 (GND_3), IC2.C15 (GND_5), IC2.C5 (GND_4), IC2.D12 (GND_7), IC2.D2 (GND_6), IC2.E9 (GND_8), IC2.F10 (GND_10), IC2.F16 (GND_11), IC2.F6 (GND_9), IC2.F8 (VCCBATT_0), IC2.G13 (GND_14), IC2.G3 (GND_12), IC2.G7 (GNDADC_0), IC2.G9 (GND_13), IC2.H6 (GND_15), IC2.H7 (VREFN_0), IC2.H8 (VP_0), IC2.J11 (GND_17), IC2.J7 (VN_0), IC2.J8 (VREFP_0), IC2.J9 (GND_16), IC2.K14 (GND_20), IC2.K4 (GND_18), IC2.K6 (GND_19), IC2.L1 (GND_21), IC2.L11 (GND_22), IC2.M10 (M1_0), IC2.M11 (M2_0), IC2.M8 (GND_23), IC2.N15 (GND_25), IC2.N5 (GND_24), IC2.P12 (GND_27), IC2.P2 (GND_26), IC2.R9 (GND_28), IC2.T16 (GND_30), IC2.T6 (GND_29), J5.1, J5.11, J5.13, J5.3, J5.5, J5.7, J5.9, J7.1, J7.13, J7.14, J7.21, J7.22, J7.23, J7.29, J7.3, J7.36, J7.5, J7.6, J7.7, L11.1, U18.10 (GND), U18.19 (*OE), U20.10 (GND), U20.19 (*OE), U21.4 (VSS), U22.2 (-VIN), U22.4 (-VOUT), Y2.2 (GND)
- net BLUE: now also R100.2, R101.2
- net GREEN: now also R116.2, R117.2
- net HSYNC: now also IC2.R15 (IO_L9P_T1_DQS_14), R115.2, U20.6 (A5)
- net RED: now also R107.2, R108.2
- net VSYNC: now also IC2.R13 (IO_L16P_T2_CSI_B_14), R114.2, U20.7 (A6)
- new net: R114.1, U20.13 (B6)
- new net: R115.1, U20.14 (B5)
- new net: R116.1, U20.15 (B4)
- new net: R118.1, U20.16 (B3)
- new net: R120.1, U20.17 (B2)
- new net: R122.1, U20.18 (B1)
- new net: R113.1, U18.18 (B1)
- new net: R112.1, R113.2
- new net: R107.1, U18.15 (B4)
- new net: R106.1, U18.14 (B5)
- new net: R105.1, R106.2
- new net: J5.6, R126.2
- new net: R110.1, R111.2, R112.2
- new net: R108.1, R109.2, R110.2
- new net: R104.1, U18.13 (B6)
- new net: R103.1, R104.2, R105.2
- new net: IC2.J3 (IO_L21P_T3_DQS_35), U15. (A20)
- new net: IC2.K1 (IO_L22P_T3_35), U15. (A20)
- new net: IC2.K2 (IO_L24N_T3_35), U15.1 (LB#)
- new net: IC2.J5 (IO_L19P_T3_35), U15.2 (OE#)
- new net: IC2.J1 (IO_L22N_T3_35), U15.3 (A0)
- new net: R101.1, R102.2, R103.2
- new net: R119.1, R120.2, R121.2
- new net: R117.1, R118.2, R119.2
- new net: J7.2, U22.6 (+VOUT)
- new net: J7.S1 (SHIELD), J7.S2 (SHIELD)
- new net: R121.1, R122.2
- new net: L11.2, U22.1 (+VIN)
- new net: R125.2, U21.7 (HOLD#/IO3/R#)
- new net: R100.1, U18.11 (B8)
- new net: R102.1, U18.12 (B7)
- new net: R109.1, U18.16 (B3)
- new net: R111.1, U18.17 (B2)
- new net: IC2.H10 (DONE_0), R94.2
- new net: J5.4, R127.2
- new net: R124.2, U21.1 (CS#)
- new net: R123.2, U21.3 (WP#/IO2)
- new net B0: IC2.T9 (IO_L22P_T3_A05_D21_14), U18.6 (A5)
- new net B1: IC2.T8 (IO_L21N_T3_DQS_A06_D22_14), U18.7 (A6)
- new net B2: IC2.T7 (IO_L21P_T3_DQS_14), U18.8 (A7)
- new net B3: IC2.T5 (IO_L23N_T3_A02_D18_14), U18.9 (A8)
- new net G0: IC2.T4 (IO_L9P_T1_DQS_34), U20.2 (A1)
- new net G1: IC2.T3 (IO_L9N_T1_DQS_34), U20.3 (A2)
- new net G2: IC2.T2 (IO_L8N_T1_34), U20.4 (A3)
- new net G3: IC2.R16 (IO_L9N_T1_DQS_D13_14), U20.5 (A4)
- new net K12: IC2.K12 (IO_0_14), U19. (A20)
- new net K13: IC2.K13 (IO_L5P_T0_D06_14), U19. (A20)
- new net L12: IC2.L12 (IO_L6P_T0_FCS_B_14), U19. (A20)
- new net L13: IC2.L13 (IO_L5N_T0_D07_14), U19. (A20)
- new net L14: IC2.L14 (IO_L4P_T0_D04_14), U19. (A20)
- new net L15: IC2.L15 (IO_L3P_T0_DQS_PUDC_B_14), U19. (A20)
- new net M14: IC2.M14 (IO_L4N_T0_D05_14), U19. (A20)
- new net M15: IC2.M15 (IO_L3N_T0_DQS_EMCCLK_14), U19. (A20)
- new net M16: IC2.M16 (IO_L7P_T1_D09_14), U19. (A20)
- new net M4: IC2.M4 (IO_L1N_T0_34), U19. (A20)
- new net M5: IC2.M5 (IO_L6P_T0_34), U19. (A20)
- new net M6: IC2.M6 (IO_L19P_T3_A10_D26_14), U19. (A20)
- new net MCU_CS: IC2.H12 (IO_L20P_T3_A20_15)
- new net MCU_MISO: IC2.H16 (IO_L22P_T3_A17_15)
- new net MCU_MOSI: IC2.H14 (IO_L24P_T3_RS1_15)
- new net MCU_SCK: IC2.H13 (IO_L20N_T3_A19_15)
- new net N1: IC2.N1 (IO_L4P_T0_34), U19.3 (A0)
- new net N11: IC2.N11 (IO_L13P_T2_MRCC_14), U19. (A20)
- new net N12: IC2.N12 (IO_L13N_T2_MRCC_14), U19. (A20)
- new net N13: IC2.N13 (IO_L11P_T1_SRCC_14), U19. (A20)
- new net N14: IC2.N14 (IO_L12P_T1_MRCC_14), U19. (A20)
- new net N16: IC2.N16 (IO_L7N_T1_D10_14), U19. (A20)
- new net N2: IC2.N2 (IO_L3N_T0_DQS_34), U19.2 (OE#)
- new net N3: IC2.N3 (IO_L3P_T0_DQS_34), U19.1 (LB#)
- new net N9: IC2.N9 (IO_L18P_T2_A12_D28_14), U19. (A20)
- new net P1: IC2.P1 (IO_L4N_T0_34), U19. (A20)
- new net P10: IC2.P10 (IO_L14P_T2_SRCC_14), U19. (A20)
- new net P11: IC2.P11 (IO_L14N_T2_SRCC_14), U19. (A20)
- new net P13: IC2.P13 (IO_L11N_T1_SRCC_14), U19. (A20)
- new net P14: IC2.P14 (IO_L12N_T1_MRCC_14), U19. (A20)
- new net P15: IC2.P15 (IO_L8P_T1_D11_14), U19. (A20)
- new net P16: IC2.P16 (IO_L8N_T1_D12_14), U19. (A20)
- new net P3: IC2.P3 (IO_L5N_T0_34), U19. (A20)
- new net P4: IC2.P4 (IO_L5P_T0_34), U19. (A20)
- new net P5: IC2.P5 (IO_L10P_T1_34), U19. (A20)
- new net P6: IC2.P6 (IO_25_14), U19. (A20)
- new net P8: IC2.P8 (IO_L20P_T3_A08_D24_14), U19. (A20)
- new net P9: IC2.P9 (IO_L18N_T2_A11_D27_14), U19. (A20)
- new net R0: IC2.T15 (IO_L10N_T1_D15_14), U18.2 (A1)
- new net R1: IC2.R1 (IO_L7N_T1_34), IC2.T14 (IO_L10P_T1_D14_14), U18.3 (A2), U19. (A20)
- new net R10: IC2.R10 (IO_L17P_T2_A14_D30_14), U19. (A20)
- new net R11: IC2.R11 (IO_L17N_T2_A13_D29_14), U19. (A20)
- new net R12: IC2.R12 (IO_L15P_T2_DQS_RDWR_B_14), U19. (A20)
- new net R2: IC2.R2 (IO_L7P_T1_34), IC2.T13 (IO_L16N_T2_A15_D31_14), U18.4 (A3), U19. (A20)
- new net R3: IC2.R3 (IO_L8P_T1_34), IC2.T10 (IO_L22N_T3_A04_D20_14), U18.5 (A4), U19. (A20)
- new net R5: IC2.R5 (IO_L23P_T3_A03_D19_14), U19. (A20)
- new net R6: IC2.R6 (IO_L24P_T3_A01_D17_14), U19. (A20)
- new net R7: IC2.R7 (IO_L24N_T3_A00_D16_14), U19. (A20)
- new net R8: IC2.R8 (IO_L20N_T3_A07_D23_14), U19. (A20)
- no-connect marks 22 -> 24
Other:
- note added: "VGA_B3 VGA_B2 VGA_B1 VGA_B0"
- note added: "VGA_G3 VGA_G2 VGA_G1 VGA_G0"
- note added: "VGA_R3 VGA_R2 VGA_R1 VGA_R0"
- note removed: "Mangler å lage en connector"
- note removed: "VGA_B0 VGA_B1 VGA_B2 VGA_B3"
- note removed: "VGA_G0 VGA_G1 VGA_G2 VGA_G3"
- note removed: "VGA_R0 VGA_R1 VGA_R2 VGA_R3"
- moved on the sheet: C1, C10, C11, C12, C13, C14, C15, C16, C17, C18, C19, C2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

Commit message: commit melding
Parts:
- removed C132: 100n, symbol Device:C
- removed R123, R125: 4.7k, symbol Device:R
- removed R124: 2.4k, symbol Device:R
- added C40, C41: 100n, symbol Device:C
- added D1: IR26-21C_L110_TR8, LED_SMD:LED_1206_3216Metric, symbol LED:IR26-21C_L110_TR8
- added R1, R3, R5, R6: 4.7k, symbol Device:R
- added R2: 2.4k, symbol Device:R
- added R4: 100, symbol Device:R
- added U1: ~, symbol S25FL127S:S25FL127S
- R94: value 330 -> 200
Connections:
- net +3.3V: now also R5.2, R6.2
- net +3V3: now also C40.1, R1.1, R2.1, R3.1, U1.8 (VCC); no longer U21.8 (VCC)
- net +5V: now also C40.2, D1.1 (K), U1.4 (VSS); no longer U21.4 (VSS)
- net at U15. (A20): now also IC2.L3 (IO_L23P_T3_35)
- net at J7.10: now also IC2.C11 (IO_L11P_T1_SRCC_15)
- net at J7.11: now also IC2.C9 (IO_L1N_T0_AD0N_15)
- net at J7.12: now also IC2.C8 (IO_L1P_T0_AD0P_15)
- net at J7.15: now also IC2.B16 (IO_L10N_T1_AD11N_15)
- net at J7.16: now also IC2.B15 (IO_L9P_T1_DQS_AD3P_15)
- net at J7.17: now also IC2.B14 (IO_L8N_T1_AD10N_15)
- net at J7.18: now also IC2.B12 (IO_L5P_T0_AD9P_15)
- net at J7.19: now also IC2.B11 (IO_L4N_T0_15)
- net at J7.20: now also IC2.B10 (IO_L4P_T0_15)
- net at J7.24: now also IC2.B9 (IO_L3P_T0_DQS_AD1P_15)
- net at J7.25: now also IC2.A15 (IO_L9N_T1_DQS_AD3N_15)
- net at J7.26: now also IC2.A14 (IO_L7N_T1_AD2N_15)
- net at J7.27: now also IC2.A13 (IO_L7P_T1_AD2P_15)
- net at J7.28: now also IC2.A12 (IO_L5N_T0_AD9N_15)
- net at J7.30: now also IC2.A10 (IO_L3N_T0_DQS_AD1N_15)
- net at J7.31: now also IC2.A9 (IO_L2N_T0_AD8N_15)
- net at J7.34: now also IC2.A8 (IO_L2P_T0_AD8P_15)
- net at J7.8: now also IC2.C13 (IO_L12N_T1_MRCC_15)
- net at J7.9: now also IC2.C12 (IO_L11N_T1_SRCC_15)
- net K16: now reaches U21.7 (HOLD#/IO3/R#)
- net K16: now also IC2.K16 (IO_L2N_T0_D03_14)
- net at IC2.H10 (DONE_0), R94.2: now also R4.2
- net at IC2.B1 (IO_L9N_T1_DQS_AD7N_35): now also U15. (A20)
- net at IC2.B2 (IO_L8P_T1_AD14P_35): now also U15. (A20)
- net at IC2.B4 (IO_L4P_T0_35): now also U15. (A20)
- net at IC2.B5 (IO_L2N_T0_AD12N_35): now also U15. (A20)
- net at IC2.B6 (IO_L2P_T0_AD12P_35): now also U15. (A20)
- net at IC2.B7 (IO_L1P_T0_AD4P_35): now also U15. (A20)
- net at IC2.C1 (IO_L9P_T1_DQS_AD7P_35): now also U15. (A20)
- net at IC2.C2 (IO_L7N_T1_AD6N_35): now also U15. (A20)
- net at IC2.C3 (IO_L7P_T1_AD6P_35): now also U15. (A20)
- net at IC2.C4 (IO_L12N_T1_MRCC_35): now also U15. (A20)
- net at IC2.C6 (IO_L5N_T0_AD13N_35): now also U15. (A20)
- net at IC2.C7 (IO_L5P_T0_AD13P_35): now also U15. (A20)
- net at IC2.D1 (IO_L10N_T1_AD15N_35): now also U15. (A20)
- net at IC2.D3 (IO_L11N_T1_SRCC_35): now also U15. (A20)
- net at IC2.D4 (IO_L12P_T1_MRCC_35): now also U15. (A20)
- net at IC2.D6 (IO_L6P_T0_35): now also U15. (A20)
- net at IC2.E1 (IO_L15N_T2_DQS_35): now also U15. (A20)
- net at IC2.E2 (IO_L10P_T1_AD15P_35): now also U15. (A20)
- net at IC2.E3 (IO_L11P_T1_SRCC_35): now also U15. (A20)
- net at IC2.E5 (IO_L13N_T2_MRCC_35): now also U15. (A20)
- net at IC2.E6 (IO_0_35): now also U15. (A20)
- net E8: now reaches IC2.E8 (CCLK_0)
- net E8: now also U21.6 (CLK)
- net at IC2.F2 (IO_L15P_T2_DQS_35): now also U15. (A20)
- net at IC2.F3 (IO_L14N_T2_SRCC_35): now also U15. (A20)
- net at IC2.F4 (IO_L14P_T2_SRCC_35): now also U15. (A20)
- net at IC2.F5 (IO_L13P_T2_MRCC_35): now also U15. (A20)
- net at IC2.G1 (IO_L17N_T2_35): now also U15. (A20)
- net at IC2.G2 (IO_L17P_T2_35): now also U15. (A20)
- net at IC2.G4 (IO_L16N_T2_35): now also U15. (A20)
- net at IC2.G5 (IO_L16P_T2_35): now also U15. (A20)
- net at IC2.H1 (IO_L20N_T3_35): now also U15. (A20)
- net at IC2.H2 (IO_L20P_T3_35): now also U15. (A20)
- net at IC2.H3 (IO_L21N_T3_DQS_35): now also U15. (A20)
- net at IC2.H4 (IO_L18N_T2_35): now also U15. (A20)
- net at IC2.H5 (IO_L18P_T2_35): now also U15. (A20)
- net J13: now reaches IC2.J13 (IO_L1P_T0_D00_MOSI_14)
- net J13: now also U21.5 (SI/IO0)
- net J14: now reaches IC2.J14 (IO_L1N_T0_D01_DIN_14)
- net J14: now also U21.2 (SO/IO1)
- net K10: now reaches IC2.K10 (INIT_B_0)
- net K10: now also R6.1
- net K15: now reaches IC2.K15 (IO_L2P_T0_D02_14)
- net K15: now also U21.3 (WP#/IO2)
- net at IC2.K3 (IO_L24P_T3_35): now also U15. (A20)
- net at IC2.K5 (IO_25_35): now also U15. (A20)
- net at IC2.L2 (IO_L23N_T3_35): now also U15. (A20)
- net L9: now reaches IC2.L9 (PROGRAM_B_0)
- net L9: now also R5.1
- net T12: now reaches IC2.T12 (IO_L15N_T2_DQS_DOUT_CSO_B_14)
- net T12: now also U21.1 (CS#)
- new net: R1.2, U1.3 (WP#/IO2)
- new net: C41.1, U21.8 (VCC)
- new net: C41.2, U21.4 (VSS)
- new net: D1.2 (A), R4.1
- new net: R3.2, U1.7 (HOLD#/IO3/R#)
- new net: R2.2, U1.1 (CS#)
Other:
- moved on the sheet: C144, J7, L11, R94, U15, U22

Commit message: commit melding
Parts:
- removed R2: 2.4k, symbol Device:R
- removed R3: 4.7k, symbol Device:R
- removed U1: ~, symbol S25FL127S:S25FL127S
- added C62, C63, C64, C65, C66, C67, C68: 470n, symbol Device:C
- added C69, C70, C71: 47u, symbol Device:C_Polarized_US
- added C72, C73, C74, C75: 4.7u, symbol Device:C
- added C76, C77, C78: 100n, symbol Device:C
- added R13, R14: 100, symbol Device:R
- C40: value 100n -> 470n
- R1: value 4.7k -> 100
- U15, U19: value ~ -> IS66WVE4M16EBLL-70BLI
Connections:
- net +3V3: now also R126.2, R127.2, U15. (A20), C62.1, C63.1, C64.1, C65.1, C66.1, C67.1, C68.1, C69.1, C70.1, C71.1, C72.1, C73.1, C74.1, C75.1, C76.2, C77.1; no longer R1.1, R126.1, R127.1
- net +5V: now also U15. (A20), C62.2, C63.2, C64.2, C65.2, C66.2, C67.2, C68.2, C69.2, C70.2, C71.2, C72.2, C73.2, C74.2, C75.2, C76.1, C77.2
- net J13: now also R13.2; no longer IC2.J13 (IO_L1P_T0_D00_MOSI_14)
- net J14: now also R1.1; no longer IC2.J14 (IO_L1N_T0_D01_DIN_14)
- net K16: now also R14.1; no longer IC2.K16 (IO_L2N_T0_D03_14)
- net MCU_CS: now also U7.31 (PA7)
- net MCU_MISO: now also U7.23 (PA1)
- net MCU_MOSI: now also U7.24 (PA2)
- net MCU_SCK: now also U7.30 (PA6)
- net at R1.2: now also IC2.J14 (IO_L1N_T0_D01_DIN_14)
- net at J5.6: now also IC2.L7 (TCK_0), R126.1; no longer R126.2
- net at Y2.3 (OUT): now also IC2.E11 (IO_L14P_T2_SRCC_15)
- net at J5.4: now also IC2.M7 (TMS_0), R127.1; no longer R127.2
- net at IC2.A7 (IO_L1N_T0_AD4N_35): now also U15. (A20)
- net at IC2.N7 (TDI_0): now also J5.10
- net at IC2.N8 (TDO_0): now also J5.8
- new net: C78.1, U19. (A20)
- new net: C78.2, U19. (A20)
- new net: IC2.K16 (IO_L2N_T0_D03_14), R14.2
- new net: IC2.J13 (IO_L1P_T0_D00_MOSI_14), R13.1
- no-connect marks 24 -> 77
Other:
- note added: "VCCO (34,35)"
- moved on the sheet: C1, C10, C11, C12, C13, C14, C141, C15, C16, C17, C18, C19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
