File: Full_schematic.kicad_sch (KiCad schematic)
At the start: 217 parts, among them IC1 XC7A100T-1FTG256C, J1 FFC3B11-40-T, J3 Conn_ST_STDC14, J5 USB_B_Micro, U1 2S7A_0518S1U, U10 MC14511BDG, U11 MAN72A, U12 MC14511BDG, U13 STM32U545VETxQ, U14 MAN72A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

Commit message: Added footprints for connectors and oscillators
Parts:
- J2: footprint Jumper:Jumper_Harwin_S1621_P10.9mm -> debug_FPGA:CONN14_877591414_MOL
- J3: footprint Jumper:Jumper_Harwin_S1621_P10.9mm -> Connector_PinHeader_1.27mm:PinHeader_2x07_P1.27mm_Vertical_SMD
- J4: footprint Jumper:Jumper_Harwin_S1621_P10.9mm -> SD_card_conn:AMPHENOL_10067847-001RLF
- U3: footprint KiCad:FH12A40S05SH55 -> TPS54294PWP:PWP16_2P31X2P46
- Y1: footprint WW100:XTAL_ASV-100.000MHZ-EC-T -> Oscillator:Oscillator_SMD_SiT_PQFN-4Pin_7.0x5.0mm
- Y2: footprint WW100:XTAL_ASV-100.000MHZ-EC-T -> Crystal:Crystal_SMD_2520-4Pin_2.5x2.0mm
Changed lines of the file:
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@@
 			)
 		)
-		(property "Footprint" "KiCad:FH12A40S05SH55"
+		(property "Footprint" "TPS54294PWP:PWP16_2P31X2P46"
 			(at 120.65 764.54 0)
 			(effects
@@
 			)
 		)
-		(property "Footprint" "Jumper:Jumper_Harwin_S1621_P10.9mm"
+		(property "Footprint" "SD_card_conn:AMPHENOL_10067847-001RLF"
 			(at 919.48 610.87 0)
 			(effects
@@
 			)
 		)
-		(property "Footprint" "WW100:XTAL_ASV-100.000MHZ-EC-T"
+		(property "Footprint" "Crystal:Crystal_SMD_2520-4Pin_2.5x2.0mm"
 			(at 604.52 516.89 0)
 			(effects
@@
 			)
 		)
-		(property "Footprint" "WW100:XTAL_ASV-100.000MHZ-EC-T"
+		(property "Footprint" "Oscillator:Oscillator_SMD_SiT_PQFN-4Pin_7.0x5.0mm"
 			(at 95.25 242.57 0)
 			(effects
@@
 			)
 		)
-		(property "Footprint" "Jumper:Jumper_Harwin_S1621_P10.9mm"
+		(property "Footprint" "Connector_PinHeader_1.27mm:PinHeader_2x07_P1.27mm_Vertical_SMD"
 			(at 789.94 567.69 0)
 			(effects
@@
 			)
 		)
-		(property "Footprint" "Jumper:Jumper_Harwin_S1621_P10.9mm"
+		(property "Footprint" "debug_FPGA:CONN14_877591414_MOL"
 			(at 420.37 194.31 0)
 			(effects

Commit message: gitty comitty
Parts:
- U2, U6: footprint IS66WVE4M16EBLL-70BLI:TFBGA48_ISI -> CY6215EV:SOP80P1184X119-44N
Connections:
- net +3V3: now also IC1.A6 (VCCO_35_1), IC1.E4 (VCCO_35_4), IC1.J2 (VCCO_35_6)
- no-connect marks 119 -> 116

Commit message: hippity gititty
Parts:
- added J6: AHDF15A-KG-TAXB, vgaaaaaa:CONN_AHDF15A-KG-TAXB_ASM, symbol vga-pin:AHDF15A-KG-TAXB
Connections:
- net BLUE: now also J6.3
- net GND: now also J6.10, J6.4, J6.5, J6.6, J6.7, J6.8, J6.9
- net GREEN: now also J6.2
- net HSYNC: now also J6.13
- net RED: now also J6.1
- net VSYNC: now also J6.14
