File: FPGA.kicad_sch (KiCad schematic)
At the start: 2 parts, among them IC1 XC7A100T-1FTG256C, Y1 ASCO

Commit message: Basic FPGA schematic
Parts:
- added C1: 330u, symbol Device:C_Polarized_US
- added C10, C11, C12, C13, C14, C15, C17, C18, C22, C23, C24, C32, C33, C34, C35, C36, C37, C38, C39, C8, C9: 470n, symbol Device:C
- added C16: 100u, symbol Device:C_Polarized_US
- added C19, C25, C26, C27: 47u, symbol Device:C_Polarized_US
- added C2, C20, C21, C28, C29, C3, C30, C31, C4, C5, C6, C7: 4.7u, symbol Device:C
- added C40, C41: 100n, symbol Device:C
- added J1: ~, symbol FPGA_Debug:FPGA_debug
- added R1, R3: 4.7k, symbol Device:R
- added R2: 2.4k, symbol Device:R
- added R4, R5: 10k, symbol Device:R
- added R6: 330, symbol Device:R
- added U1: ~, symbol S25FL127S:S25FL127S
Connections:
- net +3V3: now reaches Y1.1 (Tri-State)
- net +3V3: now also IC1.A16 (VCCO_15_1), IC1.B13 (VCCO_15_2), IC1.C10 (VCCO_15_3), IC1.E14 (VCCO_15_4), IC1.H15 (VCCO_15_5), IC1.J12 (VCCO_15_6), IC1.L16 (VCCO_14_1), IC1.L6 (VCCO_0), IC1.L7 (TCK_0), IC1.M13 (VCCO_14_2), IC1.N10 (VCCO_14_3), IC1.P7 (VCCO_14_4), IC1.R14 (VCCO_14_5), IC1.T11 (VCCO_14_6), Y1.4 (VDD), C25.1, C26.1, C27.1, C28.1, C29.1, C30.1, C31.1, C32.1, C33.1, C34.1, C35.1, C36.1, C37.1, C38.1, C39.1, C40.1, C41.1, J1.2, R1.1, R2.1, R3.1, R4.1, R5.1, R6.1, U1.8 (VCC)
- net GND: now reaches Y1.2 (GND)
- net GND: now also IC1.A1 (GND_1), IC1.A11 (GND_2), IC1.B8 (GND_3), IC1.C15 (GND_5), IC1.C5 (GND_4), IC1.D12 (GND_7), IC1.D2 (GND_6), IC1.E9 (GND_8), IC1.F10 (GND_10), IC1.F16 (GND_11), IC1.F6 (GND_9), IC1.F8 (VCCBATT_0), IC1.G13 (GND_14), IC1.G3 (GND_12), IC1.G7 (GNDADC_0), IC1.G9 (GND_13), IC1.H6 (GND_15), IC1.H7 (VREFN_0), IC1.H8 (VP_0), IC1.J11 (GND_17), IC1.J7 (VN_0), IC1.J8 (VREFP_0), IC1.J9 (GND_16), IC1.K14 (GND_20), IC1.K4 (GND_18), IC1.K6 (GND_19), IC1.L1 (GND_21), IC1.L11 (GND_22), IC1.M10 (M1_0), IC1.M11 (M2_0), IC1.M8 (GND_23), IC1.N15 (GND_25), IC1.N5 (GND_24), IC1.P12 (GND_27), IC1.P2 (GND_26), IC1.R9 (GND_28), IC1.T16 (GND_30), IC1.T6 (GND_29), C1.2, C10.2, C11.2, C12.2, C13.2, C14.2, C15.2, C16.2, C17.2, C18.2, C19.2, C2.2, C20.2, C21.2, C22.2, C23.2, C24.2, C25.2, C26.2, C27.2, C28.2, C29.2, C3.2, C30.2, C31.2, C32.2, C33.2, C34.2, C35.2, C36.2, C37.2, C38.2, C39.2, C4.2, C40.2, C41.2, C5.2, C6.2, C7.2, C8.2, C9.2, J1.1, J1.11, J1.13, J1.3, J1.5, J1.7, J1.9, U1.4 (VSS)
- net at Y1.3 (OUT): now also IC1.N11 (IO_L13P_T2_MRCC_14)
- net +1V0: now reaches IC1.E10 (VCCBRAM_1)
- net +1V0: now also IC1.F11 (VCCBRAM_2), IC1.F7 (VCCINT_1), IC1.F9 (VCCINT_2), IC1.G6 (VCCINT_3), IC1.H9 (VCCINT_4), IC1.J6 (VCCINT_5), IC1.L8 (VCCINT_7), C1.1, C10.1, C11.1, C12.1, C13.1, C14.1, C15.1, C16.1, C17.1, C18.1, C2.1, C3.1, C4.1, C5.1, C6.1, C7.1, C8.1, C9.1
- net at IC1.E8 (CCLK_0): now also U1.6 (CLK)
- net +1V8: now reaches IC1.G10 (VCCAUX_1)
- net +1V8: now also IC1.G8 (VCCADC_0), IC1.J10 (VCCAUX_2), IC1.K11 (VCCAUX_3), IC1.L10 (VCCAUX_4), C19.1, C20.1, C21.1, C22.1, C23.1, C24.1
- net at IC1.H10 (DONE_0): now also R6.2
- net at IC1.J13 (IO_L1P_T0_D00_MOSI_14): now also U1.5 (SI/IO0)
- net at IC1.K15 (IO_L2P_T0_D02_14): now also R1.2, U1.3 (WP#/IO2)
- net at IC1.K16 (IO_L2N_T0_D03_14): now also R3.2, U1.7 (HOLD#/IO3/R#)
- net at IC1.L12 (IO_L6P_T0_FCS_B_14): now also U1.2 (SO/IO1)
- net at IC1.N7 (TDI_0): now also J1.10
- net at IC1.N8 (TDO_0): now also J1.8
- new net: J1.4, R4.2
- new net: J1.6, R5.2
- new net: R2.2, U1.1 (CS#)
- no-connect marks 0 -> 2
Other:
- note added: "S25FL127S"
- note added: "U1"
- note added: "VCCAUX"
- note added: "VCCBRAM"
- note added: "VCCINT"
- note added: "VCCO (14,15)"

Commit message: schematic for stm32u545
Parts:
- renumbered C40 to C32, C41 to C33, C39 to C34, C15 to C35, C38 to C36, C14 to C37, C37 to C38, C13 to C39, C36 to C40, C12 to C41, C35 to C42, C11 to C43, C34 to C44, C10 to C45, C24 to C46, C33 to C47, C9 to C48, C23 to C49, C32 to C50, C8 to C51, C22 to C52, C26 to C53, C1 to C54, C16 to C55, C19 to C56, C25 to C57, C27 to C58, C17 to C59, C2 to C60, C20 to C61, C28 to C62, C3 to C63, C18 to C64, C21 to C65, C29 to C66, C4 to C67, C30 to C68, C5 to C69, C31 to C70, C6 to C71, C7 to C72, J1 to J5, R1 to R55, R2 to R56, R3 to R57, R6 to R58, R5 to R59, R4 to R60, U1 to U6, Y1 to Y2

Commit message: updated footprints
Parts:
- R55, R56, R57, R58, R59, R60: footprint (none) -> Resistor_SMD:R_0805_2012Metric
Changed lines of the file:
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@@
 			)
 		)
-		(property "Footprint" ""
+		(property "Footprint" "Resistor_SMD:R_0805_2012Metric"
 			(at 57.912 41.91 90)
 			(effects
@@
 			)
 		)
-		(property "Footprint" ""
+		(property "Footprint" "Resistor_SMD:R_0805_2012Metric"
 			(at 70.612 41.91 90)
 			(effects
@@
 			)
 		)
-		(property "Footprint" ""
+		(property "Footprint" "Resistor_SMD:R_0805_2012Metric"
 			(at 224.79 347.218 90)
 			(effects
@@
 			)
 		)
-		(property "Footprint" ""
+		(property "Footprint" "Resistor_SMD:R_0805_2012Metric"
 			(at 387.35 288.798 90)
 			(effects
@@
 			)
 		)
-		(property "Footprint" ""
+		(property "Footprint" "Resistor_SMD:R_0805_2012Metric"
 			(at 109.982 41.91 90)
 			(effects
@@
 			)
 		)
-		(property "Footprint" ""
+		(property "Footprint" "Resistor_SMD:R_0805_2012Metric"
 			(at 392.43 290.068 90)
 			(effects
