File: MCU.kicad_sch (KiCad schematic)
At the start: 17 parts, among them J1 Conn_ST_STDC14, SW1 SW_Nidec_CAS-120A1, U3 STM32F745VGH6, Y1 8MHz

Commit message: schematic for stm32u545
Parts:
- renumbered C30 to C21, C29 to C22, C28 to C23, C20 to C27, C27 to C28, C21 to C29, C23 to C30, C22 to C31, J1 to J4, R11 to R53, R10 to R54, U3 to U5
Changed lines of the file:
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@@
 		(dnp no)
 		(fields_autoplaced yes)
-		(property "Reference" "C28"
+		(property "Reference" "C23"
 			(at 147.32 71.1199 0)
 			(effects
@@
 			(project ""
 				(path "/071102f3-276b-4b6b-8738-8c534a30b197/4b4b82c0-0ab9-449d-bd70-557960532ad7"
-					(reference "C28")
+					(reference "C23")
 					(unit 1)
 				)
@@
 		(dnp no)
 		(fields_autoplaced yes)
-		(property "Reference" "#PWR011"
+		(property "Reference" "#PWR029"
 			(at 313.69 91.44 0)
 			(effects
@@
 			(project ""
 				(path "/071102f3-276b-4b6b-8738-8c534a30b197/4b4b82c0-0ab9-449d-bd70-557960532ad7"
-					(reference "#PWR011")
+					(reference "#PWR029")
 					(unit 1)
 				)
@@
 		(dnp no)
 		(fields_autoplaced yes)
-		(property "Reference" "C30"
+		(property "Reference" "C21"
 			(at 120.65 71.1199 0)
 			(effects
@@
 			(project "TDT4295"
 				(path "/071102f3-276b-4b6b-8738-8c534a30b197/4b4b82c0-0ab9-449d-bd70-557960532ad7"
-					(reference "C30")
+					(reference "C21")
 					(unit 1)
 				)
@@
 		(dnp no)
 		(fields_autoplaced yes)
-		(property "Reference" "#PWR08"
+		(property "Reference" "#PWR021"
 			(at 144.78 138.43 0)
 			(effects
@@
 			(project ""
 				(path "/071102f3-276b-4b6b-8738-8c534a30b197/4b4b82c0-0ab9-449d-bd70-557960532ad7"
-					(reference "#PWR08")
+					(reference "#PWR021")
 					(unit 1)
 				)
@@
 		(dnp no)
 		(fields_autoplaced yes)
-		(property "Reference" "#PWR09"
+		(property "Reference" "#PWR022"
 			(at 144.78 205.74 0)
 			(effects
@@
 			(project ""
 				(path "/071102f3-276b-4b6b-8738-8c534a30b197/4b4b82c0-0ab9-449d-bd70-557960532ad7"
-					(reference "#PWR09")
+					(reference "#PWR022")
 					(unit 1)
 				)
@@
 		(dnp no)
 		(fields_autoplaced yes)
-		(property "Reference" "C29"
+		(property "Reference" "C22"
 			(at 134.62 71.1199 0)
 			(effects
@@
 			(project "TDT4295"
 				(path "/071102f3-276b-4b6b-8738-8c534a30b197/4b4b82c0-0ab9-449d-bd70-557960532ad7"
-					(reference "C29")
+					(reference "C22")
 					(unit 1)
 				)
@@
 		(dnp no)
 		(fields_autoplaced yes)
-		(property "Reference" "#PWR014"
+		(property "Reference" "#PWR023"
 			(at 161.29 66.04 0)
 			(effects
@@
 			(project ""
 				(path "/071102f3-276b-4b6b-8738-8c534a30b197/4b4b82c0-0ab9-449d-bd70-557960532ad7"
-					(reference "#PWR014")
+					(reference "#PWR023")
 					(unit 1)
 				)
@@
 		(on_board yes)
 		(dnp no)
-		(property "Reference" "C23"
+		(property "Reference" "C30"
 			(at 243.84 179.324 0)
 			(effects
@@
 			(project "TDT4295"
 				(path "/071102f3-276b-4b6b-8738-8c534a30b197/4b4b82c0-0ab9-449d-bd70-557960532ad7"
-					(reference "C23")
+					(reference "C30")
 					(unit 1)
 				)
@@
 		(dnp no)
 		(fields_autoplaced yes)
-		(property "Reference" "U3"
+		(property "Reference" "U5"
 			(at 283.21 46.99 0)
 			(effects
@@
 			(project ""
 				(path "/071102f3-276b-4b6b-8738-8c534a30b197/4b4b82c0-0ab9-449d-bd70-557960532ad7"
-					(reference "U3")
+					(reference "U5")
 					(unit 1)
 				)
@@
 		(dnp no)
 		(fields_autoplaced yes)
-		(property "Reference" "#PWR012"
+		(property "Reference" "#PWR028"
 			(at 287.02 203.2 0)
 			(effects
@@
 			(project ""
 				(path "/071102f3-276b-4b6b-8738-8c534a30b197/4b4b82c0-0ab9-449d-bd70-557960532ad7"
-					(reference "#PWR012")
+					(reference "#PWR028")
 					(unit 1)
 				)
@@
 		(dnp no)
 		(fields_autoplaced yes)
-		(property "Reference" "R11"
+		(property "Reference" "R53"
 			(at 219.71 187.96 90)
 			(effects
@@
 			(project ""
 				(path "/071102f3-276b-4b6b-8738-8c534a30b197/4b4b82c0-0ab9-449d-bd70-557960532ad7"
-					(reference "R11")
+					(reference "R53")
 					(unit 1)
 				)
@@
 		(dnp no)
 		(fields_autoplaced yes)
-		(property "Reference" "C21"
+		(property "Reference" "C29"
 			(at 213.36 134.6199 0)
 			(effects
@@
 			(project ""
 				(path "/071102f3-276b-4b6b-8738-8c534a30b197/4b4b82c0-0ab9-449d-bd70-557960532ad7"
-					(reference "C21")
+					(reference "C29")
 					(unit 1)
 				)
@@
 		(dnp no)
 		(fields_autoplaced yes)
-		(property "Reference" "J1"
+		(property "Reference" "J4"
 			(at 133.35 166.3699 0)
 			(effects
@@
 			(project ""
 				(path "/071102f3-276b-4b6b-8738-8c534a30b197/4b4b82c0-0ab9-449d-bd70-557960532ad7"
-					(reference "J1")
+					(reference "J4")
 					(unit 1)
 				)
@@
 		(dnp no)
 		(fields_autoplaced yes)
-		(property "Reference" "R10"
+		(property "Reference" "R54"
 			(at 243.84 165.0999 0)
 			(effects
@@
 			(project ""
 				(path "/071102f3-276b-4b6b-8738-8c534a30b197/4b4b82c0-0ab9-449d-bd70-557960532ad7"
-					(reference "R10")
+					(reference "R54")
 					(unit 1)
 				)
@@
 		(dnp no)
 		(fields_autoplaced yes)
-		(property "Reference" "#PWR010"
+		(property "Reference" "#PWR027"
 			(at 200.66 149.86 0)
 			(effects
@@
 			(project ""
 				(path "/071102f3-276b-4b6b-8738-8c534a30b197/4b4b82c0-0ab9-449d-bd70-557960532ad7"
-					(reference "#PWR010")
+					(reference "#PWR027")
 					(unit 1)
 				)
@@
 		(dnp no)
 		(fields_autoplaced yes)
-		(property "Reference" "#PWR015"
+		(property "Reference" "#PWR026"
 			(at 185.42 208.28 0)
 			(effects
@@
 			(project "TDT4295"
 				(path "/071102f3-276b-4b6b-8738-8c534a30b197/4b4b82c0-0ab9-449d-bd70-557960532ad7"
-					(reference "#PWR015")
+					(reference "#PWR026")
 					(unit 1)
 				)
@@
 		(dnp no)
 		(fields_autoplaced yes)
-		(property "Reference" "#PWR013"
+		(property "Reference" "#PWR024"
 			(at 161.29 87.63 0)
 			(effects
@@
 			(project "TDT4295"
 				(path "/071102f3-276b-4b6b-8738-8c534a30b197/4b4b82c0-0ab9-449d-bd70-557960532ad7"
-					(reference "#PWR013")
+					(reference "#PWR024")
 					(unit 1)
 				)
@@
 		(dnp no)
 		(fields_autoplaced yes)
-		(property "Reference" "C22"
+		(property "Reference" "C31"
 			(at 331.47 168.9099 0)
 			(effects
@@
 			(project ""
 				(path "/071102f3-276b-4b6b-8738-8c534a30b197/4b4b82c0-0ab9-449d-bd70-557960532ad7"
-					(reference "C22")
+					(reference "C31")
 					(unit 1)
 				)
@@
 		(dnp no)
 		(fields_autoplaced yes)
-		(property "Reference" "C20"
+		(property "Reference" "C27"
 			(at 195.58 134.6199 0)
 			(effects
@@
 			(project ""
 				(path "/071102f3-276b-4b6b-8738-8c534a30b197/4b4b82c0-0ab9-449d-bd70-557960532ad7"
-					(reference "C20")
+					(reference "C27")
 					(unit 1)
 				)
@@
 		(dnp no)
 		(fields_autoplaced yes)
-		(property "Reference" "#PWR016"
+		(property "Reference" "#PWR025"
 			(at 185.42 191.77 0)
 			(effects
@@
 			(project "TDT4295"
 				(path "/071102f3-276b-4b6b-8738-8c534a30b197/4b4b82c0-0ab9-449d-bd70-557960532ad7"
-					(reference "#PWR016")
+					(reference "#PWR025")
 					(unit 1)
 				)
@@
 		(dnp no)
 		(fields_autoplaced yes)
-		(property "Reference" "C27"
+		(property "Reference" "C28"
 			(at 201.93 71.1199 0)
 			(effects
@@
 			(project "TDT4295"
 				(path "/071102f3-276b-4b6b-8738-8c534a30b197/4b4b82c0-0ab9-449d-bd70-557960532ad7"
-					(reference "C27")
-					(unit 1)
-				)
+					(reference "C28")
+					(unit 1)
+				)

Commit message: updated footprints
Parts:
- R53, R54: footprint (none) -> Resistor_SMD:R_0805_2012Metric
Changed lines of the file:
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@@
 			)
 		)
-		(property "Footprint" ""
+		(property "Footprint" "Resistor_SMD:R_0805_2012Metric"
 			(at 219.71 196.088 90)
 			(effects
@@
 			)
 		)
-		(property "Footprint" ""
+		(property "Footprint" "Resistor_SMD:R_0805_2012Metric"
 			(at 239.522 166.37 90)
 			(effects
