File: STM32U5.kicad_sch (KiCad schematic)
At the start: 26 parts, among them J6 Conn_ST_STDC14, U7 STM32U545VETxQ, Y3 48MHz

Commit message: updated footprints
Parts:
- R61, R62, R63, R64, R65: footprint (none) -> Resistor_SMD:R_0805_2012Metric
Changed lines of the file:
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@@
 			)
 		)
-		(property "Footprint" ""
+		(property "Footprint" "Resistor_SMD:R_0805_2012Metric"
 			(at 256.032 157.48 90)
 			(effects
@@
 			)
 		)
-		(property "Footprint" ""
+		(property "Footprint" "Resistor_SMD:R_0805_2012Metric"
 			(at 253.492 157.48 90)
 			(effects
@@
 			)
 		)
-		(property "Footprint" ""
+		(property "Footprint" "Resistor_SMD:R_0805_2012Metric"
 			(at 250.952 157.48 90)
 			(effects
@@
 			)
 		)
-		(property "Footprint" ""
+		(property "Footprint" "Resistor_SMD:R_0805_2012Metric"
 			(at 149.86 118.618 90)
 			(effects
@@
 			)
 		)
-		(property "Footprint" ""
+		(property "Footprint" "Resistor_SMD:R_0805_2012Metric"
 			(at 258.572 157.48 90)
 			(effects

Commit message: Fixed schematic comments
Parts:
- removed C75, C76, C77, C78, C80, C81: 100n, symbol Device:C
- removed C79: 10u, symbol Device:C
- removed C82: 2.2u, symbol Device:C
- added C84, C85, C86, C88, C96: 100n, Capacitor_SMD:C_0805_2012Metric, symbol Device:C
- added C92, C93: 2.2u, Capacitor_SMD:C_0805_2012Metric, symbol Device:C
- added C97: 0.1uF, Capacitor_SMD:C_0805_2012Metric, symbol Device:C
- added C99: 10u, Capacitor_SMD:C_0805_2012Metric, symbol Device:C
- added J8: ~, Jumper:Jumper_Harwin_S1621_P10.9mm, symbol XC7A100T-1FTG256C:SD_card_pinout
- added R81 (x2), R82 (x2), R83, R84: 10K, Resistor_SMD:R_0805_2012Metric, symbol Device:R
- C73, C87: footprint (none) -> Capacitor_SMD:C_0805_2012Metric
- C74: value 100n -> 10u; footprint (none) -> Capacitor_SMD:C_0805_2012Metric
- C80: renamed from C88; footprint (none) -> Capacitor_SMD:C_0805_2012Metric
- C82: renamed from C89; footprint (none) -> Capacitor_SMD:C_0805_2012Metric
- C83: value 2.2u -> 100n; footprint (none) -> Capacitor_SMD:C_0805_2012Metric
- C89: renamed from C86; footprint (none) -> Capacitor_SMD:C_0805_2012Metric
- C94: renamed from C85; footprint (none) -> Capacitor_SMD:C_0805_2012Metric
- C95: renamed from C84; footprint (none) -> Capacitor_SMD:C_0805_2012Metric
- J6: footprint (none) -> Jumper:Jumper_Harwin_S1621_P10.9mm
- L5: footprint (none) -> Inductor_SMD:L_0805_2012Metric
- R61: value 47 -> 10k
- R65: value 10k -> 47
- Y3: footprint (none) -> Valve:Valve_EURO
- renumbered U7 to U13
Connections:
- net VDD is gone; now on net +3.3V: U13.100 (VDD), U13.11 (VDD), U13.27 (VDD), U13.47 (VDDSMPS), U13.51 (VDD), U13.6 (VBAT), U13.75 (VDD)
- net +3.3V: now also C83.1, C87.1, C94.1, C95.1, U13.21 (VDDA), U13.73 (VDDUSB), C84.1, C85.1, C86.1, C88.1, C96.1, C99.1; no longer C73.1
- net GND: now also C73.1, C87.2, R61.1, C84.2, C85.2, C86.2, C88.2, C92.2, C93.2, C96.2, C97.2, C99.2, J8.10 (CD/GND), J8.11 (EP), J8.6 (VSS); no longer C73.2, C87.1, R65.1, U13.10 (VSS), U13.19 (VSSA), U13.26 (VSS), U13.48 (VSSSMPS), U13.50 (VSS), U13.74 (VSS), U13.99 (VSS)
- net at L5.2, U13.49 (VDD11), U13.98 (VDD11): now also C92.1, C93.1; no longer C83.1
- net MCU_PC2: now reaches U13.17 (PC2)
- net MCU_PC3: now reaches U13.18 (PC3)
- net at C89.2, U13.20 (VREF+): now also C73.2; no longer C87.2
- net MCU_MISO: now reaches U13.23 (PA1)
- net MCU_MOSI: now reaches U13.24 (PA2)
- net MCU_SCK: now reaches U13.30 (PA6)
- net MCU_CS: now reaches U13.31 (PA7)
- net MCU_PE9: now reaches U13.37 (PE9)
- net MCU_PE10: now reaches U13.38 (PE10)
- net MCU_PE11: now reaches U13.39 (PE11)
- net MCU_PB13: now reaches U13.52 (PB13)
- net MCU_PB14: now reaches U13.53 (PB14)
- net MCU_PB15: now reaches U13.54 (PB15)
- net MCU_PD9: now reaches U13.55 (PD8)
- net MCU_PD9: now also U13.56 (PD9)
- net MCU_PD10: now reaches U13.57 (PD10)
- net MCU_PD11: now reaches U13.58 (PD11)
- net MCU_PD12: now reaches U13.59 (PD12)
- net MCU_PD13: now reaches U13.60 (PD13)
- net MCU_PD14: now reaches U13.61 (PD14)
- net MCU_PD15: now reaches U13.62 (PD15)
- net MCU_PC6: now reaches U13.63 (PC6)
- net MCU_PC7: now reaches U13.64 (PC7)
- net MCU_PC8: now reaches U13.65 (PC8)
- net CS(Acitive low): now reaches U13.66 (PC9)
- net CS(Acitive low): now also J8. (CD/DATA3), R82.2
- net MCU_PA8: now reaches U13.67 (PA8)
- net MCU_PA9: now reaches U13.68 (PA9)
- net at U13.72 (PA13): now also R63.1; no longer R62.1
- net at U13.76 (PA14): now also R62.1; no longer R61.1
- net at R64.1: now also U13.89 (PB3); no longer U13.77 (PA15)
- net SCK: now reaches U13.78 (PC10)
- net SCK: now also J8.5 (CLK)
- net MISO: now reaches U13.79 (PC11)
- net MISO: now also J8.7 (DATA0), R82.2
- net MOSI: now reaches U13.80 (PC12)
- net MOSI: now also J8.3 (CMD), J8.4 (VDD), R81.2
- net at U13.94 (PH3): now also R61.2; no longer R65.2
- net at J6.8 (JTDO/SWO): now also R64.2; no longer R63.2
- net at R62.2: now also J6.6 (JCLK/SWCLK); no longer J6.4 (JTMS/SWDIO)
- net at J6.10 (JTDI/NC): now also R65.2; no longer R64.2
- new net: J8.1 (DATA2), R83.2
- new net: J8.8 (DATA1), R81.2
- new net: U13.10 (VSS), U13.26 (VSS), U13.50 (VSS), U13.74 (VSS), U13.99 (VSS)
- new net: R65.1, U13.77 (PA15)
- new net: J6.4 (JTMS/SWDIO), R63.2
- new net +3V3: C97.1, R81.1, R81.1, R82.1, R82.1, R83.1, R84.1
- new net Card Detect(Active low): J8.9 (CD), R84.2
- no-connect marks 4 -> 48
Other:
- moved on the sheet: C80, C82, C89, C94, C95, U13
