File: Full_schematic.kicad_pcb (KiCad board)
At the start: 8 copper layers, 215 x 178.7 mm, 215 parts, among them IC1 XC7A100T-1FTG256C, J1 FFC3B11-40-T, J3 Conn_ST_STDC14, J5 USB_B_Micro, J6 AHDF15A-KG-TAXB, U1 2S7A_0518S1U, U10 MC14511BDG, U11 MAN72A, U12 MC14511BDG, U13 STM32U545VETxQ, U14 MAN72A, U15 MC14511BDG, U16 MAN72A, U17 MC14511BDG, U18 PTS645SM43SMTR92LFS, U19 PTS645SM43SMTR92LFS, U2 IS66WVE4M16EBLL-70BLI, U3 TPS54294PWP, U4 TPS54325PWPR, U5 SN74ALVC245PWR, U6 IS66WVE4M16EBLL-70BLI, U7 S25FL127S, U8 SN74ALVC245PWR, U9 MAN72A, Y1 100Hz, Y2 48MHz

Commit message: gitty committy
Parts:
- moved C62 14.8 mm to (180.8, 213.9)
- moved C64 2.62 mm to (180.8, 200.4)
Connections:
- U3 pad V: (no net) -> GND
Routing:
- net GND: track 329.3 -> 324.8 mm, vias 119 -> 118
- added copper zone on F.Cu, net GND
Changed lines of the file:
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@@
 	(footprint "Capacitor_SMD:C_0805_2012Metric"
 		(layer "F.Cu")
-		(at 186.622999 200.396267 -90)
+		(at 180.8 213.95 -90)
 		(descr "Capacitor SMD 0805 (2012 Metric), square (rectangular) end terminal, IPC-7351 nominal, (Body size source: IPC-SM-782 page 76, https://www.pcb-3d.com/wordpress/wp-content/uploads/ipc-sm-782a_amendment_1_and_2.pdf, https://docs.google.com/spreadsheets/d/1BsfQQcO9C6DZCsRaXUlFlo91Tg2WpOkGARC1WS5S8t0/edit?usp=sharing), generated with kicad-footprint-generator")
 		(tags "capacitor")
@@
 			(layers "*.Cu" "*.Mask")
 			(remove_unused_layers no)
+			(net 64 "GND")
 		)
 		(pad "V" thru_hole circle
@@
 			(layers "*.Cu" "*.Mask")
 			(remove_unused_layers no)
+			(net 64 "GND")
 		)
 		(pad "V" thru_hole circle
@@
 			(layers "*.Cu" "*.Mask")
 			(remove_unused_layers no)
+			(net 64 "GND")
 		)
 		(pad "V" thru_hole circle
@@
 			(layers "*.Cu" "*.Mask")
 			(remove_unused_layers no)
+			(net 64 "GND")
 		)
 		(pad "V" thru_hole circle
@@
 			(layers "*.Cu" "*.Mask")
 			(remove_unused_layers no)
+			(net 64 "GND")
 		)
 		(pad "V" thru_hole circle
@@
 			(layers "*.Cu" "*.Mask")
 			(remove_unused_layers no)
+			(net 64 "GND")
 		)
 		(embedded_fonts no)
@@
 	(footprint "Capacitor_SMD:C_0805_2012Metric"
 		(layer "F.Cu")
-		(at 183.422999 200.396267 -90)
+		(at 180.8 200.399 -90)
 		(descr "Capacitor SMD 0805 (2012 Metric), square (rectangular) end terminal, IPC-7351 nominal, (Body size source: IPC-SM-782 page 76, https://www.pcb-3d.com/wordpress/wp-content/uploads/ipc-sm-782a_amendment_1_and_2.pdf, https://docs.google.com/spreadsheets/d/1BsfQQcO9C6DZCsRaXUlFlo91Tg2WpOkGARC1WS5S8t0/edit?usp=sharing), generated with kicad-footprint-generator")
 		(tags "capacitor")
@@
 	)
 	(segment
-		(start 183.422999 199.446267)
-		(end 183.422999 198.348266)
+		(start 180.8 199.449)
+		(end 180.8 198.350999)
 		(width 0.2)
 		(layer "F.Cu")
@@
 	)
 	(segment
-		(start 186.622999 199.446267)
-		(end 186.622999 198.248266)
+		(start 180.8 213)
+		(end 180.8 211.801999)
 		(width 0.2)
 		(layer "F.Cu")
@@
 	)
 	(via
-		(at 183.422999 198.348266)
+		(at 180.8 198.350999)
 		(size 0.6)
 		(drill 0.3)
@@
 	)
 	(via
-		(at 186.622999 198.248266)
+		(at 180.8 211.801999)
 		(size 0.6)
 		(drill 0.3)
@@
 	)
 	(segment
-		(start 163.3 206.9)
-		(end 163.2 206.8)
-		(width 0.2)
-		(layer "F.Cu")
-		(net 64)
-	)
-	(segment
 		(start 157.400001 151.176105)
 		(end 157.400001 151.178106)
@@
 	)
 	(segment
-		(start 163.3 206.9)
-		(end 163.670966 207.270966)
-		(width 0.2)
-		(layer "F.Cu")
-		(net 64)
-	)
-	(segment
 		(start 218.725 146.406105)
 		(end 218.725 147.231105)
@@
 	)
 	(segment
-		(start 183.422999 201.346267)
-		(end 183.422999 202.448266)
+		(start 180.8 201.349)
+		(end 180.8 202.450999)
 		(width 0.2)
 		(layer "F.Cu")
@@
 	)
 	(segment
-		(start 163.2 206.8)
-		(end 162.2 206.8)
-		(width 0.2)
-		(layer "F.Cu")
-		(net 64)
-	)
-	(segment
 		(start 273.1 91.376105)
 		(end 273.1 92.650701)
@@
 	)
 	(segment
-		(start 164.320977 207.920977)
-		(end 163.3 206.9)
-		(width 0.2)
-		(layer "F.Cu")
-		(net 64)
-	)
-	(segment
 		(start 156.400001 150.176105)
 		(end 156.385994 150.176105)
@@
 	)
 	(segment
-		(start 186.622999 201.346267)
-		(end 186.622999 202.548266)
+		(start 180.8 214.9)
+		(end 180.8 216.101999)
 		(width 0.2)
 		(layer "F.Cu")
@@
 	)
 	(segment
-		(start 163.670966 207.270966)
-		(end 163.670966 208.718267)
-		(width 0.2)
-		(layer "F.Cu")
-		(net 64)
-	)
-	(segment
 		(start 231.2 95.078105)
 		(end 231.163199 95.114906)
@@
 	)
 	(via
-		(at 183.422999 202.448266)
+		(at 180.8 202.450999)
 		(size 0.6)
 		(drill 0.3)
@@
 	)
 	(via
-		(at 186.622999 202.548266)
+		(at 180.8 216.101999)
 		(size 0.6)
 		(drill 0.3)
@@
 	)
 	(via
-		(at 162.2 206.8)
-		(size 0.6)
-		(drill 0.3)
-		(layers "F.Cu" "B.Cu")
-		(net 64)
-	)
-	(via
 		(at 168.5 134.476105)
 		(size 0.6)
@@
 	)
 	(segment
-		(start 164.320977 203.899289)
-		(end 164.320977 202.876267)
-		(width 0.2)
-		(layer "F.Cu")
-		(net 75)
-	)
-	(segment
-		(start 164.022999 204.197267)
-		(end 164.320977 203.899289)
-		(width 0.2)
-		(layer "F.Cu")
-		(net 75)
-	)
-	(segment
 		(start 179.867305 208.076105)
 		(end 181.2 208.076105)
@@
 	)
 	(via
-		(at 164.022999 204.197267)
+		(at 163.900366 200.699634)
 		(size 0.6)
 		(drill 0.3)
@@
 	)
 	(segment
-		(start 167.951841 208.126109)
-		(end 164.022999 204.197267)
+		(start 172.4 208.126109)
+		(end 171.326841 208.126109)
+		(width 0.2)
+		(layer "In5.Cu")
+		(net 75)
+	)
+	(segment
+		(start 171.326841 208.126109)
+		(end 163.900366 200.699634)
 		(width 0.2)
 		(layer "In5.Cu")
@@
 	(segment
 		(start 179.719001 208.126109)
-		(end 167.951841 208.126109)
+		(end 172.4 208.126109)
 		(width 0.2)
 		(layer "In5.Cu")
@@
 	)
 	(zone
+		(net 64)
+		(net_name "GND")
+		(layer "F.Cu")
+		(hatch edge 0.5)
+		(priority 2)
+		(connect_pads yes
+			(clearance 0.5)
+		)
+		(min_thickness 0.25)
+		(filled_areas_thickness no)
+		(fill yes
+			(thermal_gap 0.5)
+			(thermal_bridge_width 0.5)
+		)
+		(polygon
+			(pts
+				(xy 182.7 196.2) (xy 185.6 196.2) (xy 185.6 215.5) (xy 182.7 215.5)
+			)
+		)
+	)
+	(zone
+		(net 64)
+		(net_name "GND")
+		(layer "F.Cu")
+		(hatch edge 0.5)
+		(priority 2)
+		(connect_pads yes
+			(clearance 0.5)
+		)
+		(min_thickness 0.25)
+		(filled_areas_thickness no)
+		(fill yes
+			(thermal_gap 0.5)
+			(thermal_bridge_width 0.5)
+		)
+		(polygon
+			(pts
+				(xy 170.3 207.2) (xy 162.4 207.2) (xy 159.1 210) (xy 156 210) (xy 156 207) (xy 159.1 207) (xy 162.4 204.4)
+				(xy 170.3 204.4)
+			)
+		)
+	)
+	(zone
