File: Full_schematic.kicad_pcb (KiCad board)
At the start: 8 copper layers, 215 x 178.7 mm, 215 parts, among them IC1 XC7A100T-1FTG256C, J1 FFC3B11-40-T, J3 Conn_ST_STDC14, J5 USB_B_Micro, J6 AHDF15A-KG-TAXB, U1 2S7A_0518S1U, U10 MC14511BDG, U11 MAN72A, U12 MC14511BDG, U13 STM32U545VETxQ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

Commit message: fix power under FPGA
Connections:
- IC1 pad A7: unconnected-(IC1-IO_L1N_T0_AD4N_35-PadA7) -> A2
Routing:
- net +1V0: track 101.9 -> 124.4 mm
- net +3V3: track 171.6 -> 186.5 mm
- net +1V8: track 72.3 -> 79.4 mm
- added copper zone on In6.Cu, net Net-(J5-VBUS)

Commit message: add half of jumpers
Parts:
- added REF**: AMPHENOL_G800W306018EU, G800W306018EU:AMPHENOL_G800W306018EU, F.Cu at (218.0, 207.0)
- added REF**: AMPHENOL_G800W306018EU, G800W306018EU:AMPHENOL_G800W306018EU, F.Cu at (203.8, 197.7)
- added REF**: AMPHENOL_G800W306018EU, G800W306018EU:AMPHENOL_G800W306018EU, F.Cu at (214.3, 196.3)
- added REF**: AMPHENOL_G800W306018EU, G800W306018EU:AMPHENOL_G800W306018EU, F.Cu at (210.4, 205.5)
- moved C62 15.2 mm to (187.8, 200.5)
Connections:
- IC1 pad A5: unconnected-(IC1-IO_L3P_T0_DQS_AD5P_35-PadA5) -> VSYNC2
- IC1 pad A7: A2 -> HSYNC2
- J1 pad 32: unconnected-(J1-Pad32) -> HSYNC2
- J1 pad 33: unconnected-(J1-Pad33) -> VSYNC2
- U11 pad 14: +3.3V -> +3V3
- U11 pad 3: +3.3V -> +3V3
- U14 pad 14: +3.3V -> +3V3
- U14 pad 3: +3.3V -> +3V3
- U16 pad 14: +3.3V -> +3V3
- U16 pad 3: +3.3V -> +3V3
- U9 pad 14: +3.3V -> +3V3
- U9 pad 3: +3.3V -> +3V3
Routing:
- net VSYNC2: track 0.00 -> 75.7 mm
- net HSYNC2: track 0.00 -> 75.2 mm
- net GND: track 324.8 -> 359.0 mm, vias 118 -> 125
- net +3.3V: track 46.7 -> 51.0 mm, vias 12 -> 13
- net Net-(IC1-IO_L2P_T0_AD8P_15): track 74.9 -> 75.6 mm

Commit message: gittyy comitty
Parts:
- moved REF** 37.9 mm to (174.5, 193.2)
- moved REF** 12.4 mm to (191.5, 196.1)
Connections:
- C62 pad 1: +3V3 -> +3.3V
- C64 pad 1: +3V3 -> +3.3V
- L4 pad 2: +3V3 -> +3.3V
- R9 pad 1: +3V3 -> +3.3V
- REF** pad 1: (no net) -> +3.3V
- REF** pad 2: (no net) -> +3V3
- REF** pad 1: (no net) -> +1V8
- REF** pad 2: (no net) -> +1V8
Routing:
- net GND: track 359.0 -> 402.3 mm
- net +1V8: track 79.4 -> 70.0 mm, vias 10 -> 11
- net +3V3: track 186.5 -> 181.6 mm, vias 60 -> 56
- net +3.3V: track 51.0 -> 55.8 mm, vias 13 -> 17
- added copper zone on In3.Cu, net +3.3V

Commit message: Heatsinks ++
Parts:
- moved R12 0.68 mm to (157.9, 157.0)
Routing:
- net Net-(J5-VBUS): track 151.2 -> 164.9 mm
- net GND: track 402.3 -> 400.4 mm, vias 125 -> 170
- net K10: track 2.71 -> 2.08 mm
- net Net-(U3-EN2): track 18.3 -> 19.0 mm
- net CS(Acitive low): track 99.8 -> 100.3 mm
- net Net-(U4-VBST): track 4.31 -> 4.25 mm, vias 1 -> 0
- net (no net): vias 2 -> 0
- removed copper zone on In3.Cu, net Net-(J5-VBUS)
